Commit message: [modify]add urdf gps frame

File: urdf/backpack_2d.urdf (robot description, URDF)
Before this commit: robot cartographer_backpack_2d, 4 links, 3 joints
Links:
- removed link vertical_laser_link
- added link gps; visual cylinder length=0.05 radius=0.03
Joints:
- removed joint vertical_laser_link_joint
- added joint gps_joint: type fixed, parent base_link, child gps, origin xyz=0.1007 0 0.1814 rpy=0 -1.570796 3.141593
