Commit message: fix urdf

File: urdf/robot_model.urdf (robot description, URDF)
Before this commit: robot robot_model, 2 links, 1 joints
Links:
- link base_link: geometry visual box size=1.0 0.700 0.500
Joints:
- joint laser_joint: origin xyz=0 0 0.05 rpy=0 0 3.1415926 -> xyz=0.3 0 0.30 rpy=0 0 3.1415926

Commit message: change lidar pose

File: urdf/robot_model.urdf (robot description, URDF)
Before this commit: robot robot_model, 2 links, 1 joints
Joints:
- joint laser_joint: origin xyz=0.3 0 0.30 rpy=0 0 3.1415926 -> xyz=-0.3 0 0.05 rpy=0 0 3.1415926
